Commit message: updated dimensions

File: zebROS_ws/src/frcrobot_description/four_bar_elevator_2023/urdf/four_bar_ex.xacro (robot description, xacro)
@@ -2,12 +2,14 @@
 <robot xmlns:xacro="http://www.ros.org/wiki/xacro" name="four_bar_elevator">
     <xacro:property name="theta" value="${pi/6}"/>
-    <xacro:property name="L" value=".5"/>
+    <xacro:property name="L" value="1.2"/>
+    <xacro:property name="b" value="0.127"/>
+    <xacro:property name="h" value="0.243"/>
     <link name="base_link">
     </link>
     <link name="four_bar_base">
         <visual>
-            <origin xyz="0 0.25 0" rpy="1.57 0 0" />
+            <origin xyz="0 ${b/2} 0" rpy="${pi/2} 0 0" />
             <geometry>
-                <cylinder radius="0.02" length="0.5" />
+                <cylinder radius="0.02" length="${b}" />
             </geometry>
             <material name="blue">
@@ -16,16 +18,16 @@
         </visual>
     </link>
-    <joint name="joint0" type="revolute">
+    <joint name="four_bar" type="revolute">
         <parent link="four_bar_base"/>
         <child link="link1"/>
         <origin xyz="0 0 0" rpy="0 0 0" />
         <axis xyz="1 0 0" />
-        <limit lower="-1.57" upper="1.57" effort="0.5293" velocity="6.159937255" />
+        <limit lower="${-pi/2}" upper="${pi/2}" effort="0.5293" velocity="6.159937255" />
     </joint>
     <link name="link1">
         <visual>
-            <origin xyz="0 0 0.25" rpy="0 0 0" />
+            <origin xyz="0 0 ${h/2}" rpy="0 0 0" />
             <geometry>
-                <cylinder radius="0.02" length="0.5" />
+                <cylinder radius="0.02" length="${h}" />
             </geometry>
             <material name="yellow">
@@ -37,14 +39,14 @@
         <parent link="four_bar_base"/>
         <child link="link2"/>
-        <origin xyz="0 0.5 0" rpy="0 0 0" />
+        <origin xyz="0 ${b} 0" rpy="0 0 0" />
         <axis xyz="1 0 0" />
-        <limit lower="-1.57" upper="1.57" effort="0.5293" velocity="6.159937255" />
-        <mimic joint="joint0" multiplier="1" offset="0" />
+        <limit lower="${-pi/2}" upper="${pi/2}" effort="0.5293" velocity="6.159937255" />
+        <mimic joint="four_bar" multiplier="1" offset="0" />
     </joint>
     <link name="link2">
         <visual>
-            <origin xyz="0 0 0.25" rpy="0 0 0" />
+            <origin xyz="0 0 ${h/2}" rpy="0 0 0" />
             <geometry>
-                <cylinder radius="0.02" length="0.5" />
+                <cylinder radius="0.02" length="${h}" />
             </geometry>
             <material name="green">
@@ -56,14 +58,14 @@
         <parent link="link1"/>
         <child link="link3"/>
-        <origin xyz="0 0 0.5" rpy="0 0 0" />
+        <origin xyz="0 0 ${h}" rpy="0 0 0" />
         <axis xyz="1 0 0" />
-        <limit lower="-1.57" upper="1.57" effort="0.5293" velocity="6.159937255" />
-        <mimic joint="joint0" multiplier="-1" offset="0" />
+        <limit lower="${-pi/2}" upper="${pi/2}" effort="0.5293" velocity="6.159937255" />
+        <mimic joint="four_bar" multiplier="-1" offset="0" />
     </joint>
     <link name="link3">
         <visual>
-            <origin xyz="0 0.25 0" rpy="1.57 0 0" />
+            <origin xyz="0 ${b/2} 0" rpy="${pi/2} 0 0" />
             <geometry>
-                <cylinder radius="0.02" length="0.5" />
+                <cylinder radius="0.02" length="${b}" />
             </geometry>
             <material name="red">
@@ -83,5 +85,5 @@
         </visual>
     </link>
-    <joint name="elevator_joint" type="prismatic">
+    <joint name="elevator_leader" type="prismatic">
         <parent link="base_link"/>
         <child link="four_bar_base"/>
