Commit message: code to push

File: zebROS_ws/src/frcrobot_description/turret_2023/urdf/four_bar_ex.xacro (robot description, xacro)
@@ -1,98 +1,224 @@
 <?xml version="1.0"?>
-<robot xmlns:xacro="http://www.ros.org/wiki/xacro" name="four_bar_elevator">
-    <xacro:property name="theta" value="${pi/6}"/>
-    <xacro:property name="L" value="1.2"/>
-    <xacro:property name="b" value="0.127"/>
-    <xacro:property name="h" value="0.243"/>
-    <link name="base_link">
-    </link>
-    <link name="four_bar_base">
-        <visual>
-            <origin xyz="0 ${b/2} 0" rpy="${pi/2} 0 0" />
-            <geometry>
-                <cylinder radius="0.02" length="${b}" />
-            </geometry>
-            <material name="blue">
-                <color rgba="0 0 .8 1" />
-            </material>
-        </visual>
-    </link>
-    <joint name="four_bar" type="revolute">
-        <parent link="four_bar_base"/>
-        <child link="link1"/>
-        <origin xyz="0 0 0" rpy="0 0 0" />
-        <axis xyz="1 0 0" />
-        <limit lower="${-pi/2}" upper="${pi/2}" effort="0.5293" velocity="6.159937255" />
-    </joint>
-    <link name="link1">
-        <visual>
-            <origin xyz="0 0 ${h/2}" rpy="0 0 0" />
-            <geometry>
-                <cylinder radius="0.02" length="${h}" />
-            </geometry>
-            <material name="yellow">
-                <color rgba=".8 0 .8 1" />
-            </material>
-        </visual>
-    </link>
-    <joint name="joint1" type="revolute">
-        <parent link="four_bar_base"/>
-        <child link="link2"/>
-        <origin xyz="0 ${b} 0" rpy="0 0 0" />
-        <axis xyz="1 0 0" />
-        <limit lower="${-pi/2}" upper="${pi/2}" effort="0.5293" velocity="6.159937255" />
-        <mimic joint="four_bar" multiplier="1" offset="0" />
-    </joint>
-    <link name="link2">
-        <visual>
-            <origin xyz="0 0 ${h/2}" rpy="0 0 0" />
-            <geometry>
-                <cylinder radius="0.02" length="${h}" />
-            </geometry>
-            <material name="green">
-                <color rgba="0 .8 0 1" />
-            </material>
-        </visual>
-    </link>
-    <joint name="joint2" type="revolute">
-        <parent link="link1"/>
-        <child link="link3"/>
-        <origin xyz="0 0 ${h}" rpy="0 0 0" />
-        <axis xyz="1 0 0" />
-        <limit lower="${-pi/2}" upper="${pi/2}" effort="0.5293" velocity="6.159937255" />
-        <mimic joint="four_bar" multiplier="-1" offset="0" />
-    </joint>
-    <link name="link3">
-        <visual>
-            <origin xyz="0 ${b/2} 0" rpy="${pi/2} 0 0" />
-            <geometry>
-                <cylinder radius="0.02" length="${b}" />
-            </geometry>
-            <material name="red">
-                <color rgba=".8 0 0 1" />
-            </material>
-        </visual>
-    </link>
-    <link name="elevator">
-        <visual>
-            <origin xyz="0 ${L*sin(theta)/2} ${L*cos(theta)/2}" rpy="0 ${theta} ${pi/2}"/>
-            <geometry>
-                <cylinder radius="0.02" length="${L}"/>
-            </geometry>
-            <material name="white">
-                <color rgba="1 1 1 1"/>
-            </material>
-        </visual>
-    </link>
-    <joint name="elevator_leader" type="prismatic">
-        <parent link="base_link"/>
-        <child link="four_bar_base"/>
-        <origin xyz="0 0 0" rpy="0 0 0"/>
-        <axis xyz="0 ${theta} 1"/>
-        <limit effort="1000.0" lower="0" upper="${L}" velocity="0.5"/>
-    </joint>
-    <joint name="elevator_to_base" type="fixed">
-        <parent link="base_link"/>
-        <child link="elevator"/>
-    </joint>
+<robot xmlns:sensor="http://playerstage.sourceforge.net/gazebo/xmlschema/#sensor"
+	 xmlns:controller="http://playerstage.sourceforge.net/gazebo/xmlschema/#controller"
+	 xmlns:interface="http://playerstage.sourceforge.net/gazebo/xmlschema/#interface"
+	 xmlns:xacro="http://playerstage.sourceforge.net/gazebo/xmlschema/#interface"
+	 name="r2d2">
+	<xacro:property name="width" value=".2" />
+	<xacro:property name="leglen" value=".6" />
+	<xacro:property name="polelen" value=".2" />
+	<xacro:property name="bodylen" value=".6" />
+	<xacro:property name="baselen" value=".4" />
+	<xacro:property name="wheeldiam" value=".07" />
+	<xacro:property name="pi" value="3.1415" />
+	<xacro:macro name="default_inertial" params="mass">
+		<inertial>
+      			<mass value="${mass}" />
+		        <inertia ixx="1.0" ixy="0.0" ixz="0.0"
+			         iyy="1.0" iyz="0.0"
+			         izz="1.0" />
+		</inertial>
+	</xacro:macro>
+	<link name="base_link">
+		<visual>
+			<geometry>
+				<cylinder radius="${width}" length="${bodylen}"/>
+			</geometry>
+			<material name="blue">
+				<color rgba="0 0 .8 1"/>
+			</material>
+		</visual>
+		<collision>
+			<geometry>
+				<cylinder radius="${width}" length="${bodylen}"/>
+			</geometry>
+		</collision>
+		<xacro:default_inertial mass="10"/>
+	</link>
+	<xacro:macro name="wheel" params="prefix suffix reflect">
+		<link name="${prefix}_${suffix}_wheel">
+			<visual>
+				<geometry>
+					<cylinder radius="${wheeldiam/2}" length=".1"/>
+				</geometry>
+				<material name="black">
+					<color rgba="0 0 0 1"/>
+				</material>
+			</visual>
+			<collision>
+				<geometry>
+					<cylinder radius="${wheeldiam/2}" length=".1"/>
+				</geometry>
+			</collision>
+			<xacro:default_inertial mass="1"/>
+		</link>
+		<joint name="${prefix}_${suffix}_wheel_joint" type="continuous">
+			<axis xyz="0 0 1"/>
+			<parent link="${prefix}_base"/>
+			<child link="${prefix}_${suffix}_wheel"/>
+			<origin xyz="0 ${baselen*reflect/3} -${wheeldiam/2+.05}" rpy="0 ${pi/2} 0"/>
+      			<limit effort="100" velocity="100" />
+			<joint_properties damping="0.0" friction="0.0" />
+		</joint>
+	    <gazebo reference="${prefix}_${suffix}_wheel" >
+	      <mu1>50.0</mu1>
+	      <mu2>50.0</mu2>
+	      <kp>100000000.0</kp>
+	      <kd>1.0</kd>
+	      <material>Gazebo/Fish</material>
+	    </gazebo>
+	</xacro:macro>
+	<xacro:macro name="leg" params="prefix reflect">
+		<link name="${prefix}_leg">
+			<visual>
+				<geometry>
+					<box size="${leglen} .2 .1"/>
+				</geometry>
+				<origin xyz="0 0 -${leglen/2}" rpy="0 ${pi/2} 0"/>
+				<material name="white">
+					<color rgba="1 1 1 1"/>
+				</material>
+			</visual>
+			<collision>
+				<geometry>
+					<box size="${leglen} .2 .1"/>
+				</geometry>
+				<origin xyz="0 0 -${leglen/2}" rpy="0 ${pi/2} 0"/>
+			</collision>
+			<xacro:default_inertial mass="10"/>
+		</link>
+		<joint name="base_to_${prefix}_leg" type="fixed">
+			<parent link="base_link"/>
+			<child link="${prefix}_leg"/>
+			<origin xyz="${reflect*(width+.02)} 0 .25" />
+		</joint>
+		<link name="${prefix}_base">
+			<visual>
+				<geometry>
+					<box size=".1 ${baselen} .1"/>
+				</geometry>
+				<material name="white"/>
+			</visual>
+			<collision>
+				<geometry>
+					<box size=".1 ${baselen} .1"/>
+				</geometry>
+			</collision>
+			<xacro:default_inertial mass="10"/>
+		</link>
+		<joint name="${prefix}_base_joint" type="fixed">
+			<parent link="${prefix}_leg"/>
+			<child link="${prefix}_base"/>
+			<origin xyz="0 0 ${-leglen}" />
+		</joint>
+		<xacro:wheel prefix="${prefix}" suffix="front" reflect="1"/>
+		<xacro:wheel prefix="${prefix}" suffix="back" reflect="-1"/>
+	</xacro:macro>
+	<xacro:leg prefix="right" reflect="1" />
+	<xacro:leg prefix="left" reflect="-1" />
+	<joint name="gripper_extension" type="prismatic">
+		<parent link="base_link"/>
+		<child link="gripper_pole"/>
+    		<limit effort="1000.0" lower="-${width*2-.02}" upper="0" velocity="0.5"/>
+		<origin rpy="0 0 ${pi/2}" xyz="0 ${width-.01} .2"/>
+	</joint>
+	<link name="gripper_pole">
+		<visual>
+			<geometry>
+				<cylinder length="${polelen}" radius=".01"/>
+			</geometry>
+			<origin xyz="${polelen/2} 0 0" rpy="0 ${pi/2} 0 "/>
+		</visual>
+		<collision>
+			<geometry>
+				<cylinder length="${polelen}" radius=".01"/>
+			</geometry>
+			<origin xyz="${polelen/2} 0 0" rpy="0 ${pi/2} 0 "/>
+		</collision>
+		<xacro:default_inertial mass=".05"/>
+	</link>
+	<xacro:macro name="gripper" params="prefix reflect">
+		<joint name="${prefix}_gripper_joint" type="revolute">
+			<axis xyz="0 0 ${reflect}"/>
+			<limit effort="1000.0" lower="0.0" upper="0.548" velocity="0.5"/>
+			<origin rpy="0 0 0" xyz="${polelen} ${reflect*0.01} 0"/>
+			<parent link="gripper_pole"/>
+			<child link="${prefix}_gripper"/>
+		</joint>
+		<link name="${prefix}_gripper">
+			<visual>
+     				<origin rpy="${(reflect-1)/2*pi} 0 0" xyz="0 0 0"/>
+				<geometry>
+					<mesh filename="package://pr2_description/meshes/gripper_v0/l_finger.dae"/>
+				</geometry>
+			</visual>
+			<collision>
+				<geometry>
+					<mesh filename="package://pr2_description/meshes/gripper_v0/l_finger.dae"/>
+				</geometry>
+     				<origin rpy="${(reflect-1)/2*pi} 0 0" xyz="0 0 0"/>
+			</collision>
+			<xacro:default_inertial mass=".05"/>
+		</link>
+		<joint name="${prefix}_tip_joint" type="fixed">
+			<parent link="${prefix}_gripper"/>
+			<child link="${prefix}_tip"/>
+		</joint>
+		<link name="${prefix}_tip">
+			<visual>
+     				<origin rpy="${(reflect-1)/2*pi} 0 0" xyz="0.09137 0.00495 0"/>
+				<geometry>
+					<mesh filename="package://pr2_description/meshes/gripper_v0/l_finger_tip.dae"/>
+				</geometry>
+			</visual>
+			<collision>
+				<geometry>
+					<mesh filename="package://pr2_description/meshes/gripper_v0/l_finger_tip.dae"/>
+				</geometry>
+     				<origin rpy="${(reflect-1)/2*pi} 0 0" xyz="0.09137 0.00495 0"/>
+			</collision>
+			<xacro:default_inertial mass=".05"/>
+		</link>
+	</xacro:macro>
+	<xacro:gripper prefix="left" reflect="1" />
+	<xacro:gripper prefix="right" reflect="-1" />
+	<link name="head">
+		<visual>
+			<geometry>
+				<sphere radius="${width}"/>
+			</geometry>
+			<material name="white"/>
+		</visual>
+		<collision>
+			<geometry>
+				<sphere radius="${width}"/>
+			</geometry>
+		</collision>
+		<xacro:default_inertial mass="10"/>
+	</link>
+	<joint name="head_swivel" type="continuous">
+		<parent link="base_link"/>
+		<child link="head"/>
+		<axis xyz="0 0 1"/>
+		<origin xyz="0 0 ${bodylen/2}"/>
+	</joint>
+	<link name="box">
+		<visual>
+			<geometry>
+				<box size=".08 .08 .08"/>
+			</geometry>
+			<material name="blue"/>
+		</visual>
+		<collision>
+			<geometry>
+				<box size=".08 .08 .08"/>
+			</geometry>
+		</collision>
+		<xacro:default_inertial mass="1"/>
+	</link>
+	<joint name="tobox" type="fixed">
+		<parent link="head"/>
+		<child link="box"/>
+		<origin xyz="0 ${.707*width} ${.707*width}"/>
+	</joint>
 </robot>

File: zebROS_ws/src/frcrobot_description/turret_2023/urdf/r2d2.xacro (robot description, xacro)
@@ -16,187 +16,4 @@
       </geometry>
       <material name="blue"/>
-    </visual>
-  </link>
-  <link name="right_leg">
-    <visual>
-      <geometry>
-        <box size="0.6 0.1 0.2"/>
-      </geometry>
-      <origin rpy="0 1.57075 0" xyz="0 0 -0.3"/>
-      <material name="white"/>
-    </visual>
-  </link>
-  <joint name="base_to_right_leg" type="fixed">
-    <parent link="base_link"/>
-    <child link="right_leg"/>
-    <origin xyz="0 -0.22 0.25"/>
-  </joint>
-  <link name="right_base">
-    <visual>
-      <geometry>
-        <box size="0.4 0.1 0.1"/>
-      </geometry>
-      <material name="white"/>
-    </visual>
-  </link>
-  <joint name="right_base_joint" type="fixed">
-    <parent link="right_leg"/>
-    <child link="right_base"/>
-    <origin xyz="0 0 -0.6"/>
-  </joint>
-  <link name="right_front_wheel">
-    <visual>
-      <origin rpy="1.57075 0 0" xyz="0 0 0"/>
-      <geometry>
-        <cylinder length="0.1" radius="0.035"/>
-      </geometry>
-      <material name="black"/>
-      <origin rpy="0 0 0" xyz="0 0 0"/>
-    </visual>
-  </link>
-  <joint name="right_front_wheel_joint" type="continuous">
-    <axis rpy="0 0 0" xyz="0 1 0"/>
-    <parent link="right_base"/>
-    <child link="right_front_wheel"/>
-    <origin rpy="0 0 0" xyz="0.133333333333 0 -0.085"/>
-  </joint>
-  <link name="right_back_wheel">
-    <visual>
-      <origin rpy="1.57075 0 0" xyz="0 0 0"/>
-      <geometry>
-        <cylinder length="0.1" radius="0.035"/>
-      </geometry>
-      <material name="black"/>
-    </visual>
-  </link>
-  <joint name="right_back_wheel_joint" type="continuous">
-    <axis rpy="0 0 0" xyz="0 1 0"/>
-    <parent link="right_base"/>
-    <child link="right_back_wheel"/>
-    <origin rpy="0 0 0" xyz="-0.133333333333 0 -0.085"/>
-  </joint>
-  <link name="left_leg">
-    <visual>
-      <geometry>
-        <box size="0.6 0.1 0.2"/>
-      </geometry>
-      <origin rpy="0 1.57075 0" xyz="0 0 -0.3"/>
-      <material name="white"/>
-    </visual>
-  </link>
-  <joint name="base_to_left_leg" type="fixed">
-    <parent link="base_link"/>
-    <child link="left_leg"/>
-    <origin xyz="0 0.22 0.25"/>
-  </joint>
-  <link name="left_base">
-    <visual>
-      <geometry>
-        <box size="0.4 0.1 0.1"/>
-      </geometry>
-      <material name="white"/>
-    </visual>
-  </link>
-  <joint name="left_base_joint" type="fixed">
-    <parent link="left_leg"/>
-    <child link="left_base"/>
-    <origin xyz="0 0 -0.6"/>
-  </joint>
-  <link name="left_front_wheel">
-    <visual>
-      <origin rpy="1.57075 0 0" xyz="0 0 0"/>
-      <geometry>
-        <cylinder length="0.1" radius="0.035"/>
-      </geometry>
-      <material name="black"/>
-    </visual>
-  </link>
-  <joint name="left_front_wheel_joint" type="continuous">
-    <axis rpy="0 0 0" xyz="0 1 0"/>
-    <parent link="left_base"/>
-    <child link="left_front_wheel"/>
-    <origin rpy="0 0 0" xyz="0.133333333333 0 -0.085"/>
-  </joint>
-  <link name="left_back_wheel">
-    <visual>
-      <origin rpy="1.57075 0 0" xyz="0 0 0"/>
-      <geometry>
-        <cylinder length="0.1" radius="0.035"/>
-      </geometry>
-      <material name="black"/>
-    </visual>
-  </link>
-  <joint name="left_back_wheel_joint" type="continuous">
-    <axis rpy="0 0 0" xyz="0 1 0"/>
-    <parent link="left_base"/>
-    <child link="left_back_wheel"/>
-    <origin rpy="0 0 0" xyz="-0.133333333333 0 -0.085"/>
-  </joint>
-  <joint name="gripper_extension" type="prismatic">
-    <parent link="base_link"/>
-    <child link="gripper_pole"/>
-    <limit effort="1000.0" lower="-0.38" upper="0" velocity="0.5"/>
-    <origin rpy="0 0 0" xyz="0.19 0 0.2"/>
-  </joint>
-  <link name="gripper_pole">
-    <visual>
-      <geometry>
-        <cylinder length="0.2" radius="0.01"/>
-      </geometry>
-      <origin rpy="0 1.57075 0 " xyz="0.1 0 0"/>
-    </visual>
-  </link>
-  <joint name="left_gripper_joint" type="revolute">
-    <axis xyz="0 0 1"/>
-    <limit effort="1000.0" lower="0.0" upper="0.548" velocity="0.5"/>
-    <origin rpy="0 0 0" xyz="0.2 0.01 0"/>
-    <parent link="gripper_pole"/>
-    <child link="left_gripper"/>
-  </joint>
-  <link name="left_gripper">
-    <visual>
-      <origin rpy="0.0 0 0" xyz="0 0 0"/>
-      <geometry>
-        <mesh filename="package://urdf_tutorial/meshes/l_finger.dae"/>
-      </geometry>
-    </visual>
-  </link>
-  <joint name="left_tip_joint" type="fixed">
-    <parent link="left_gripper"/>
-    <child link="left_tip"/>
-  </joint>
-  <link name="left_tip">
-    <visual>
-      <origin rpy="0.0 0 0" xyz="0.09137 0.00495 0"/>
-      <geometry>
-        <mesh filename="package://urdf_tutorial/meshes/l_finger_tip.dae"/>
-      </geometry>
-    </visual>
-  </link>
-  <joint name="right_gripper_joint" type="revolute">
-    <axis xyz="0 0 -1"/>
-    <limit effort="1000.0" lower="0.0" upper="0.548" velocity="0.5"/>
-    <origin rpy="0 0 0" xyz="0.2 -0.01 0"/>
-    <parent link="gripper_pole"/>
-    <child link="right_gripper"/>
-  </joint>
-  <link name="right_gripper">
-    <visual>
-      <origin rpy="-3.1415 0 0" xyz="0 0 0"/>
-      <geometry>
-        <mesh filename="package://urdf_tutorial/meshes/l_finger.dae"/>
-      </geometry>
-    </visual>
-  </link>
-  <joint name="right_tip_joint" type="fixed">
-    <parent link="right_gripper"/>
-    <child link="right_tip"/>
-  </joint>
-  <link name="right_tip">
-    <visual>
-      <origin rpy="-3.1415 0 0" xyz="0.09137 0.00495 0"/>
-      <geometry>
-        <mesh filename="package://urdf_tutorial/meshes/l_finger_tip.dae"/>
-      </geometry>
     </visual>
   </link>
