Commit message: R2D2==Turret

File: zebROS_ws/src/frcrobot_description/turret_2023/urdf/turret.xacro (robot description, xacro)
@@ -11,10 +11,4 @@
   </material>
   <link name="base_link">
-    <visual>
-      <geometry>
-        <cylinder length="0.6" radius="0.2"/>
-      </geometry>
-      <material name="blue"/>
-    </visual>
   </link>
   <link name="head">
@@ -26,5 +20,5 @@
     </visual>
   </link>
-  <joint name="head_swivel" type="continuous">
+  <joint name="turret_joint" type="continuous">
     <parent link="base_link"/>
     <child link="head"/>

Commit message: turret looks cool now

File: zebROS_ws/src/frcrobot_description/turret_2023/urdf/turret.xacro (robot description, xacro)
@@ -13,10 +13,4 @@
   </link>
   <link name="head">
-    <visual>
-      <geometry>
-        <sphere radius="0.2"/>
-      </geometry>
-      <material name="white"/>
-    </visual>
   </link>
   <joint name="turret_joint" type="continuous">
@@ -24,12 +18,11 @@
     <child link="head"/>
     <axis xyz="0 0 1"/>
-    <origin xyz="0 0 0.3"/>
+    <origin xyz="0 0 0.0"/>
   </joint>
   <link name="box">
     <visual>
       <geometry>
-        <box size="0.08 0.08 0.08"/>
+        <mesh filename="package://turret_2023/meshes/CITRUS_TURRET_HOOD.dae"/>
       </geometry>
-      <material name="blue"/>
     </visual>
   </link>
@@ -37,5 +30,19 @@
     <parent link="head"/>
     <child link="box"/>
-    <origin xyz="0.1814 0 0.1414"/>
+    <origin xyz="0.0 0 0.0"/>
   </joint>
+  <joint name="to_field" type="fixed">
+    <parent link="base_link"/>
+    <child link="full_field"/>
+    <origin xyz="0.0 0 0.0"/>
+  </joint>
+  <link name="full_field">
+    <parent link="base_link"/>
+    <visual>
+      <origin rpy="0.0 0 0" xyz="0 0 0"/>
+      <geometry>
+        <mesh filename="package://turret_2023/meshes/MINIFRC_FIELD.dae"/>
+      </geometry>
+    </visual>
+  </link>
 </robot>

Commit message: update rviz file

File: zebROS_ws/src/frcrobot_description/turret_2023/urdf/turret.xacro (robot description, xacro)
@@ -46,3 +46,17 @@
     </visual>
   </link>
+  <joint name="to_robot" type="fixed">
+    <parent link="base_link"/>
+    <child link="robot_chassis"/>
+    <origin xyz="0.0 0 0.0"/>
+  </joint>
+  <link name="robot_chassis">
+    <parent link="base_link"/>
+    <visual>
+      <origin rpy="0.0 0 0" xyz="0 0 0"/>
+      <geometry>
+        <mesh filename="package://turret_2023/meshes/900_2023_NO_ELEVATOR.dae"/>
+      </geometry>
+    </visual>
+  </link>
 </robot>

Commit message: swerve drive vis support

File: zebROS_ws/src/frcrobot_description/turret_2023/urdf/turret.xacro (robot description, xacro)
@@ -46,17 +46,3 @@
     </visual>
   </link>
-  <joint name="to_robot" type="fixed">
-    <parent link="base_link"/>
-    <child link="robot_chassis"/>
-    <origin xyz="0.0 0 0.0"/>
-  </joint>
-  <link name="robot_chassis">
-    <parent link="base_link"/>
-    <visual>
-      <origin rpy="0.0 0 0" xyz="0 0 0"/>
-      <geometry>
-        <mesh filename="package://turret_2023/meshes/900_2023_NO_ELEVATOR.dae"/>
-      </geometry>
-    </visual>
-  </link>
 </robot>
