Commit message: reorganization to find packages

File: zebROS_ws/src/gazebra/chimera_description/y2023_urdf/robot.urdf (robot description, URDF)
Before this commit: robot onshape, 14 links, 13 joints
Links:
- link central_chassis: mass 7.7787891582795705148 -> 7.7787891582795740675; geometry collision mesh filename=package:///central_chassis_collision.stl; visual mesh filename=package:///central_chassis_visual.stl
- link first_stage: mass 0.37485540355657037681 -> 0.37485540355657043232; geometry collision mesh filename=package:///first_stage_collision.stl; visual mesh filename=package:///first_stage_visual.stl
- link first_stage_2: mass 0.37485540355657043232 -> 0.37485540355657048783; geometry collision mesh filename=package:///first_stage_2_collision.stl; visual mesh filename=package:///first_stage_2_visual.stl
- link first_stage_3: geometry collision mesh filename=package:///first_stage_3_collision.stl; visual mesh filename=package:///first_stage_3_visual.stl
- link first_stage_4: mass 0.37485540355657037681 -> 0.37485540355657048783; geometry collision mesh filename=package:///first_stage_4_collision.stl; visual mesh filename=package:///first_stage_4_visual.stl
- link fixed_stage: mass 2.1102377118690225366 -> 2.1102377118679833679; geometry collision mesh filename=package:///fixed_stage_collision.stl; visual mesh filename=package:///fixed_stage_visual.stl
- link fixed_stage_2: mass 2.1102377118690238689 -> 2.1102377118679847001; geometry collision mesh filename=package:///fixed_stage_2_collision.stl; visual mesh filename=package:///fixed_stage_2_visual.stl
- link fixed_stage_3: mass 2.1102377118690234248 -> 2.110237711867984256; geometry collision mesh filename=package:///fixed_stage_3_collision.stl; visual mesh filename=package:///fixed_stage_3_visual.stl
- link fixed_stage_4: mass 2.1102377118690234248 -> 2.110237711867984256; geometry collision mesh filename=package:///fixed_stage_4_collision.stl; visual mesh filename=package:///fixed_stage_4_visual.stl
- link second_stage: mass 0.34193546654456347111 -> 0.34193546654456352663; geometry collision mesh filename=package:///second_stage_collision.stl; visual mesh filename=package:///second_stage_visual.stl
- link second_stage_2: mass 0.3419354665445634156 -> 0.34193546654456352663; geometry collision mesh filename=package:///second_stage_2_collision.stl; visual mesh filename=package:///second_stage_2_visual.stl
- link second_stage_3: mass 0.34193546654456347111 -> 0.34193546654456352663; geometry collision mesh filename=package:///second_stage_3_collision.stl; visual mesh filename=package:///second_stage_3_visual.stl
- link second_stage_4: mass 0.34193546654456347111 -> 0.34193546654456352663; geometry collision mesh filename=package:///second_stage_4_collision.stl; visual mesh filename=package:///second_stage_4_visual.stl

Commit message: something is happening in gazebo involving chimera

File: zebROS_ws/src/gazebra/chimera_description/y2023_urdf/robot.urdf (robot description, URDF)
Before this commit: robot onshape, 14 links, 13 joints
Links:
- link central_chassis: geometry collision mesh filename=package://chimera_description/y2023_urdf/central_chassis_co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; visual mesh filename=package://chimera_description/y2023_urdf/central_chassis_vi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
- link first_stage: geometry collision mesh filename=package://chimera_description/y2023_urdf/first_stage_collis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; visual mesh filename=package://chimera_description/y2023_urdf/first_stage_visual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
- link first_stage_2: geometry collision mesh filename=package://chimera_description/y2023_urdf/first_stage_2_coll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; visual mesh filename=package://chimera_description/y2023_urdf/first_stage_2_visu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
- link first_stage_3: geometry collision mesh filename=package://chimera_description/y2023_urdf/first_stage_3_coll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; visual mesh filename=package://chimera_description/y2023_urdf/first_stage_3_visu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
- link first_stage_4: geometry collision mesh filename=package://chimera_description/y2023_urdf/first_stage_4_coll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; visual mesh filename=package://chimera_description/y2023_urdf/first_stage_4_visu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
- link fixed_stage: geometry collision mesh filename=package://chimera_description/y2023_urdf/fixed_stage_collis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; visual mesh filename=package://chimera_description/y2023_urdf/fixed_stage_visual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
- link fixed_stage_2: geometry collision mesh filename=package://chimera_description/y2023_urdf/fixed_stage_2_coll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; visual mesh filename=package://chimera_description/y2023_urdf/fixed_stage_2_visu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
- link fixed_stage_3: geometry collision mesh filename=package://chimera_description/y2023_urdf/fixed_stage_3_coll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; visual mesh filename=package://chimera_description/y2023_urdf/fixed_stage_3_visu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
- link fixed_stage_4: geometry collision mesh filename=package://chimera_description/y2023_urdf/fixed_stage_4_coll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; visual mesh filename=package://chimera_description/y2023_urdf/fixed_stage_4_visu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
- link second_stage: geometry collision mesh filename=package://chimera_description/y2023_urdf/second_stage_colli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; visual mesh filename=package://chimera_description/y2023_urdf/second_stage_visua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
- link second_stage_2: geometry collision mesh filename=package://chimera_description/y2023_urdf/second_stage_2_col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; visual mesh filename=package://chimera_description/y2023_urdf/second_stage_2_vis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
- link second_stage_3: geometry collision mesh filename=package://chimera_description/y2023_urdf/second_stage_3_col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; visual mesh filename=package://chimera_description/y2023_urdf/second_stage_3_vis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
- link second_stage_4: geometry collision mesh filename=package://chimera_description/y2023_urdf/second_stage_4_col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; visual mesh filename=package://chimera_description/y2023_urdf/second_stage_4_vis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
