Commit message: MOVES (very bad but still)

File: zebROS_ws/src/frcrobot_description/frcrobot_description/urdf/frcrobot.urdf (robot description, URDF)
Before this commit: robot onshape, 14 links, 13 joints
Joints:
- removed joint bl_angle
- removed joint bl_drive
- removed joint br_angle
- removed joint br_drive
- removed joint fl_angle
- removed joint fl_drive
- removed joint fr_angle
- removed joint fr_drive
- added joint left_back_angle_wheel: type continuous, parent fixed_stage_2, child first_stage_2, origin xyz=0.06667500000000003979 0.007556500000000021533 -0.019843749999999965583 rpy=1.570796326794896558 0.74446276911887487859 3.141592653589793116, axis 0 0 1, limit effort=1 velocity=20
- added joint left_back_drive_wheel: type continuous, parent first_stage_2, child second_stage_2, origin xyz=-0.014718639782431541807 -0.014718639782432388352 0.041331500000000201411 rpy=1.5707963267948981123 -0.10233292597333981666 -0.78539816339744639162, axis 0 0 1, limit effort=1 velocity=20
- added joint left_front_angle_wheel: type continuous, parent fixed_stage, child first_stage, origin xyz=0.066674999999999984279 0.0075565000000000354108 -0.019843749999999937828 rpy=-1.5707963267948954478 -0.0013042609915997001487 -9.0564346581562362991e-16, axis 0 0 1, limit effort=1 velocity=20
- added joint left_front_drive_wheel: type continuous, parent first_stage, child second_stage, origin xyz=-0.014718639782432818564 -0.014718639782432485497 0.041331499999999611605 rpy=1.5707963267948974462 0.3547103969677229407 -0.78539816339744616958, axis 0 0 1, limit effort=1 velocity=20
- added joint right_back_angle_wheel: type continuous, parent fixed_stage_3, child first_stage_3, origin xyz=-0.066293999999999908557 0.0079375000000000278666 -0.019843749999999937828 rpy=1.570796326794896558 -1.3713290209023065724 3.1415926535897726879, axis 0 0 1, limit effort=1 velocity=20
- added joint right_back_drive_wheel: type continuous, parent first_stage_3, child second_stage_3, origin xyz=-0.013550659703940370893 -0.013550659703939815781 0.041331499999998508321 rpy=-1.5707963267948952257 -0.38629807207531591251 2.3561944901923501661, axis 0 0 1, limit effort=1 velocity=20
- added joint right_front_angle_wheel: type continuous, parent fixed_stage_4, child first_stage_4, origin xyz=0.066293999999999908557 -0.0079375000000000972555 0.019843750000000076605 rpy=-1.570796326794896558 1.2358944559116720185 3.141592653589793116, axis 0 0 1, limit effort=1 velocity=20
- added joint right_front_drive_wheel: type continuous, parent first_stage_4, child second_stage_4, origin xyz=-0.014718639782432263452 -0.014718639782432541008 0.041331500000000041817 rpy=-1.5707963267948994446 0.53105430610586668028 2.3561944901923461693, axis 0 0 1, limit effort=1 velocity=20
