Commit message: attempting to make things move, inital transmission and removeing swerve drive controller

File: zebROS_ws/src/frcrobot_description/frcrobot_description/urdf/swerve_base.urdf (robot description, URDF)
Before this commit: robot onshape, 14 links, 13 joints
Joints:
- removed joint right_front_angle_wheel
- added joint elevator_leader: type continuous, parent fixed_stage_4, child first_stage_4, origin xyz=0.066293999999999908557 -0.0079375000000000972555 0.019843750000000076605 rpy=-1.570796326794896558 1.2358944559116720185 3.141592653589793116, axis 0 0 1, limit effort=1 velocity=20

Commit message: IT LIVES (also pushed like 40stls but thats a later problem)

File: zebROS_ws/src/frcrobot_description/frcrobot_description/urdf/swerve_base.urdf (robot description, URDF)
Before this commit: robot onshape, 14 links, 13 joints
Links:
- removed link first_stage_4
- removed link second_stage_4
- added link fr_angle, mass 0.37485540355657037681; collision mesh filename=package://frcrobot_description/meshes/first_stage_4_collisi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; visual mesh filename=package://frcrobot_description/meshes/first_stage_4_visual.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
- added link fr_drive, mass 0.34193546654456347111; collision mesh filename=package://frcrobot_description/meshes/second_stage_4_collis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; visual mesh filename=package://frcrobot_description/meshes/second_stage_4_visual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
Joints:
- removed joint fr_angle
- removed joint fr_drive
- added joint fr_angle_joint: type continuous, parent fixed_stage_4, child first_stage_4, origin xyz=0.066293999999999908557 -0.0079375000000000972555 0.019843750000000076605 rpy=-1.570796326794896558 1.2358944559116720185 3.141592653589793116, axis 0 0 1, limit effort=1 velocity=20
- added joint fr_drive_joint: type continuous, parent first_stage_4, child second_stage_4, origin xyz=-0.014718639782432263452 -0.014718639782432541008 0.041331500000000041817 rpy=-1.5707963267948994446 0.53105430610586668028 2.3561944901923461693, axis 0 0 1, limit effort=1 velocity=20
