Commit message: nothing works, sim torque is off, applying the correct torque in gazebo also looks wrong

File: zebROS_ws/src/frcrobot_description/frcrobot_description/urdf/robot_2023.urdf (robot description, URDF)
Before this commit: robot onshape, 14 links, 13 joints
Links:
- link bl_fixed_link: mass 2.1102377118679847001 -> 10.002377118679847001
- link br_fixed_link: mass 2.110237711867984256 -> 10.00237711867984256
- link fl_fixed_link: mass 2.1102377118679847001 -> 10.002377118679847001
- link fr_fixed_link: mass 2.1102377118679851442 -> 10.002377118679851442

Commit message: kinda works now, still need to modify post processing

File: zebROS_ws/src/frcrobot_description/frcrobot_description/urdf/robot_2023.urdf (robot description, URDF)
Before this commit: robot onshape, 14 links, 13 joints
Links:
- link bl_angle_link: mass 0.37485540355657037681 -> 0.37485540355657048783
- link bl_drive_link: mass 0.23325990258684708989 -> 0.23325990258684717316
- link bl_fixed_link: mass 10.002377118679847001 -> 2.1102377118679838119
- link br_angle_link: mass 0.37485540355657037681 -> 0.37485540355657043232
- link br_drive_link: mass 0.23325990258684708989 -> 0.23325990258684717316
- link br_fixed_link: mass 10.00237711867984256 -> 2.1102377118679833679
- link fl_angle_link: mass 0.37485540355657037681 -> 0.37485540355657043232
- link fl_drive_link: mass 0.23325990258684708989 -> 0.23325990258684717316
- link fl_fixed_link: mass 10.002377118679847001 -> 2.1102377118679838119
- link fr_angle_link: mass 0.37485540355657037681 -> 0.37485540355657048783
- link fr_drive_link: mass 0.23325990258684708989 -> 0.23325990258684717316
- link fr_fixed_link: mass 10.002377118679851442 -> 2.110237711867984256
Joints:
- joint bl_drive: origin xyz=-0.01471863978243215243 -0.014718639782432601723 0.041331499999999986306 rpy=-1.5707963267948985564 0.47976839601182080797 2.3561944901923439488 -> xyz=-0.014718639782432096919 -0.014718639782432601723 0.041331499999999986306 rpy=-1.5707963267948985564 0.47976839601182086348 2.3561944901923439488
- joint br_drive: origin xyz=-0.014718639782432386617 -0.014718639782432596519 0.041331500000000014061 rpy=1.5707963267948990005 0.56629976412908578087 -0.78539816339744417117 -> xyz=-0.014718639782432376209 -0.014718639782432596519 0.041331500000000014061 rpy=1.5707963267948990005 0.56629976412908578087 -0.78539816339744417117
- joint fl_drive: origin xyz=-0.013550659703939711698 -0.013550659703939982315 0.0413314999999997712 rpy=1.5707963267948983344 0.0066490939608964379562 -0.78539816339744317197 -> xyz=-0.013550659703939713432 -0.013550659703939982315 0.0413314999999997712 rpy=1.5707963267948983344 0.0066490939608964379562 -0.78539816339744317197
- joint fr_drive: origin xyz=-0.014718639782432374474 -0.01471863978243261907 0.041331500000000236106 rpy=1.5707963267949003328 1.2191085435220101463 -0.7853981633974378429 -> xyz=-0.014718639782432374474 -0.01471863978243261907 0.041331500000000229167 rpy=-1.5707963267948974462 -0.0045778681610583937464 2.3561944901923461693
