Commit message: we have textures now

File: zebROS_ws/src/frcrobot_description/frcrobot_description/urdf/2024_field.urdf (robot description, URDF)
Before this commit: robot field, 2 links, 1 joints
Links:
- link central_chassis: geometry visual mesh filename=package://frcrobot_description/meshes/CrescendoField.dae

Commit message: foxglove stuff

File: zebROS_ws/src/frcrobot_description/frcrobot_description/urdf/2024_field.urdf (robot description, URDF)
Before this commit: robot field, 2 links, 1 joints
Links:
- removed link base_link
- removed link central_chassis
- added link map
- added link water_game_link; visual mesh filename=package://frcrobot_description/meshes/Crescendo_Field.dae
Joints:
- removed joint base_link_to_base
- added joint map_to_base: type fixed, parent map, child water_game_link, origin xyz=0 0 0 rpy=0.0 0 0

Commit message: remove static map->odom in viz

File: zebROS_ws/src/frcrobot_description/frcrobot_description/urdf/2024_field.urdf (robot description, URDF)
Before this commit: robot field, 2 links, 1 joints
Links:
- link water_game_link: geometry visual mesh filename=package://frcrobot_description/meshes/CrescendoField.dae
