Commit message: review

File: zebROS_ws/src/minifrcrobot_description/urdf/robot.urdf (robot description, URDF)
Before this commit: robot onshape, 17 links, 16 joints
Links:
- removed link robot_code_ready_link_rio
- added link babys_first_orchestra_link
- added link candle1_link
- added link pcm_link
- added link pigeon2_link
- added link robot_code_ready_rio_link
Joints:
- added joint babys_first_orchestra: type fixed, parent base_link, child babys_first_orchestra_link, origin xyz=0 0 0 rpy=0.0 0 0
- added joint candle1: type fixed, parent base_link, child candle1_link, origin xyz=0 0 0 rpy=0.0 0 0
- added joint pcm: type fixed, parent base_link, child pcm_link, origin xyz=0 0 0 rpy=0.0 0 0
- added joint pigeon2: type fixed, parent base_link, child pigeon2_link, origin xyz=0 0 0 rpy=0.0 0 0
- joint robot_code_ready_rio: child robot_code_ready_link_rio -> robot_code_ready_rio_link

Commit message: add minifrc stls

File: zebROS_ws/src/minifrcrobot_description/urdf/robot.urdf (robot description, URDF)
Before this commit: robot onshape, 21 links, 20 joints
Links:
- removed link babys_first_orchestra_link
- removed link candle1_link
- removed link pcm_link
- removed link pigeon2_link
- removed link robot_code_ready_link
- removed link robot_code_ready_rio_link
Joints:
- removed joint babys_first_orchestra
- removed joint candle1
- removed joint pcm
- removed joint pigeon2
- removed joint robot_code_ready_jetson
- removed joint robot_code_ready_rio

Commit message: Added the controller for the arm, and started on the action server and client (Also fixed some stuff with simlaunch but yea)

File: zebROS_ws/src/minifrcrobot_description/urdf/robot.urdf (robot description, URDF)
Before this commit: robot onshape, 15 links, 14 joints
Links:
- added link pcm_link
- added link robot_code_ready_jetson_link
- added link robot_code_ready_rio_link
Joints:
- added joint pcm: type fixed, parent base_link, child pcm_link, origin xyz=0 0 0 rpy=0.0 0 0
- added joint robot_code_ready_jetson: type fixed, parent base_link, child robot_code_ready_jetson_link, origin xyz=0 0 0 rpy=0.0 0 0
- added joint robot_code_ready_rio: type fixed, parent base_link, child robot_code_ready_rio_link, origin xyz=0 0 0 rpy=0.0 0 0
